File: AMS-Mega2560-Base/file61534325.kicad_sch (KiCad schematic)
At the start: 3 parts, among them IC22 24PCDFA6D, IC23 INA849DR

Commit message: fixing some library settings and updating some schematics
Parts:
- renumbered IC22 to IC19, IC23 to IC20, R52 to R42
Connections:
- net +10V: no longer IC19.1 (VCC)
- net +2V5: no longer IC20.6 (REF)
- net +5VP: no longer IC20.8 (+VS)
- net GND: no longer IC19.3 (GROUND), IC20.5 (-VS)
- net VacOut: no longer IC20.7 (OUT)
Changed lines of the file:
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@@
 (kicad_sch (version 20211123) (generator eeschema)
   (paper "A4")
+  (wire (pts (xy 106.68 68.58) (xy 96.52 68.58))
+    (stroke (width 0) (type default) (color 0 0 0 0))
+  )
+  (wire (pts (xy 99.06 66.04) (xy 96.52 66.04))
+    (stroke (width 0) (type default) (color 0 0 0 0))
+  )
+  (wire (pts (xy 149.86 87.63) (xy 92.71 87.63))
+    (stroke (width 0) (type default) (color 0 0 0 0))
+  )
+  (wire (pts (xy 179.07 92.71) (xy 177.8 92.71))
+    (stroke (width 0) (type default) (color 0 0 0 0))
+  )
+  (wire (pts (xy 149.86 90.17) (xy 110.49 90.17))
+    (stroke (width 0) (type default) (color 0 0 0 0))
+  )
   (wire (pts (xy 177.8 90.17) (xy 193.04 90.17))
     (stroke (width 0) (type default) (color 0 0 0 0))
   )
+  (wire (pts (xy 177.8 87.63) (xy 180.34 87.63))
+    (stroke (width 0) (type default) (color 0 0 0 0))
+  )
+  (wire (pts (xy 92.71 87.63) (xy 92.71 95.25))
+    (stroke (width 0) (type default) (color 0 0 0 0))
+  )
+  (wire (pts (xy 149.86 85.09) (xy 106.68 85.09))
+    (stroke (width 0) (type default) (color 0 0 0 0))
+  )
+  (wire (pts (xy 99.06 72.39) (xy 99.06 66.04))
+    (stroke (width 0) (type default) (color 0 0 0 0))
+  )
+  (wire (pts (xy 180.34 85.09) (xy 180.34 80.01))
+    (stroke (width 0) (type default) (color 0 0 0 0))
+  )
+  (wire (pts (xy 133.35 92.71) (xy 149.86 92.71))
+    (stroke (width 0) (type default) (color 0 0 0 0))
+  )
+  (wire (pts (xy 179.07 92.71) (xy 179.07 96.52))
+    (stroke (width 0) (type default) (color 0 0 0 0))
+  )
+  (wire (pts (xy 106.68 85.09) (xy 106.68 68.58))
+    (stroke (width 0) (type default) (color 0 0 0 0))
+  )
+  (wire (pts (xy 177.8 85.09) (xy 180.34 85.09))
+    (stroke (width 0) (type default) (color 0 0 0 0))
+  )
+  (wire (pts (xy 96.52 60.96) (xy 99.06 60.96))
+    (stroke (width 0) (type default) (color 0 0 0 0))
+  )
+  (wire (pts (xy 99.06 60.96) (xy 99.06 54.61))
+    (stroke (width 0) (type default) (color 0 0 0 0))
+  )
+  (wire (pts (xy 96.52 63.5) (xy 133.35 63.5))
+    (stroke (width 0) (type default) (color 0 0 0 0))
+  )
+  (wire (pts (xy 110.49 90.17) (xy 110.49 95.25))
+    (stroke (width 0) (type default) (color 0 0 0 0))
+  )
   (wire (pts (xy 133.35 63.5) (xy 133.35 92.71))
-    (stroke (width 0) (type default) (color 0 0 0 0))
-  )
-  (wire (pts (xy 110.49 90.17) (xy 110.49 95.25))
-    (stroke (width 0) (type default) (color 0 0 0 0))
-  )
-  (wire (pts (xy 99.06 72.39) (xy 99.06 66.04))
-    (stroke (width 0) (type default) (color 0 0 0 0))
-  )
-  (wire (pts (xy 149.86 85.09) (xy 106.68 85.09))
-    (stroke (width 0) (type default) (color 0 0 0 0))
-  )
-  (wire (pts (xy 92.71 87.63) (xy 92.71 95.25))
-    (stroke (width 0) (type default) (color 0 0 0 0))
-  )
-  (wire (pts (xy 179.07 92.71) (xy 177.8 92.71))
-    (stroke (width 0) (type default) (color 0 0 0 0))
-  )
-  (wire (pts (xy 99.06 66.04) (xy 96.52 66.04))
-    (stroke (width 0) (type default) (color 0 0 0 0))
-  )
-  (wire (pts (xy 177.8 87.63) (xy 180.34 87.63))
-    (stroke (width 0) (type default) (color 0 0 0 0))
-  )
-  (wire (pts (xy 99.06 60.96) (xy 99.06 54.61))
-    (stroke (width 0) (type default) (color 0 0 0 0))
-  )
-  (wire (pts (xy 106.68 68.58) (xy 96.52 68.58))
-    (stroke (width 0) (type default) (color 0 0 0 0))
-  )
-  (wire (pts (xy 177.8 85.09) (xy 180.34 85.09))
-    (stroke (width 0) (type default) (color 0 0 0 0))
-  )
-  (wire (pts (xy 133.35 92.71) (xy 149.86 92.71))
-    (stroke (width 0) (type default) (color 0 0 0 0))
-  )
-  (wire (pts (xy 106.68 85.09) (xy 106.68 68.58))
-    (stroke (width 0) (type default) (color 0 0 0 0))
-  )
-  (wire (pts (xy 149.86 90.17) (xy 110.49 90.17))
-    (stroke (width 0) (type default) (color 0 0 0 0))
-  )
-  (wire (pts (xy 180.34 85.09) (xy 180.34 80.01))
-    (stroke (width 0) (type default) (color 0 0 0 0))
-  )
-  (wire (pts (xy 179.07 92.71) (xy 179.07 96.52))
-    (stroke (width 0) (type default) (color 0 0 0 0))
-  )
-  (wire (pts (xy 96.52 60.96) (xy 99.06 60.96))
-    (stroke (width 0) (type default) (color 0 0 0 0))
-  )
-  (wire (pts (xy 96.52 63.5) (xy 133.35 63.5))
-    (stroke (width 0) (type default) (color 0 0 0 0))
-  )
-  (wire (pts (xy 149.86 87.63) (xy 92.71 87.63))
     (stroke (width 0) (type default) (color 0 0 0 0))
   )
@@
   (symbol (lib_id "SamacSys_Parts:24PCDFA6D") (at 96.52 68.58 180)
     (in_bom yes) (on_board yes)
-    (property "Reference" "IC22" (id 0) (at 85.2932 54.229 0))
+    (property "Reference" "IC19" (id 0) (at 85.2932 54.229 0))
     (property "Value" "24PCDFA6D" (id 1) (at 85.2932 56.5404 0))
     (property "Footprint" "SamacSys_Parts:24PCDFA6D" (id 2) (at 72.39 71.12 0)
@@
       (effects (font (size 1.27 1.27)) (justify left) hide)
     )
-    (pin "1")
-    (pin "2")
-    (pin "3")
-    (pin "4")
   )
   (symbol (lib_id "SamacSys_Parts:INA849DR") (at 149.86 85.09 0)
     (in_bom yes) (on_board yes)
-    (property "Reference" "IC23" (id 0) (at 163.83 78.359 0))
+    (property "Reference" "IC20" (id 0) (at 163.83 78.359 0))
     (property "Value" "INA849DR" (id 1) (at 163.83 80.6704 0))
     (property "Footprint" "SamacSys_Parts:SOIC127P600X175-8N" (id 2) (at 173.99 82.55 0)
@@
       (effects (font (size 1.27 1.27)) (justify left) hide)
     )
-    (pin "1")
-    (pin "2")
-    (pin "3")
-    (pin "4")
-    (pin "5")
-    (pin "6")
-    (pin "7")
-    (pin "8")
   )
   (symbol (lib_id "SamacSys_Parts:YR1B665RCC") (at 92.71 95.25 0)
     (in_bom yes) (on_board yes)
-    (property "Reference" "R52" (id 0) (at 101.6 89.535 0))
+    (property "Reference" "R42" (id 0) (at 101.6 89.535 0))
     (property "Value" "YR1B665RCC" (id 1) (at 101.6 91.8464 0))
     (property "Footprint" "SamacSys_Parts:RESAD1550W60L630D230" (id 2) (at 106.68 93.98 0)
@@
       (effects (font (size 1.27 1.27)) (justify left) hide)
     )
-    (pin "1")
-    (pin "2")
   )
   (symbol (lib_id "power:+10V") (at 99.06 54.61 0)
     (in_bom yes) (on_board yes)
-    (property "Reference" "#PWR0125" (id 0) (at 99.06 58.42 0)
+    (property "Reference" "#PWR0120" (id 0) (at 99.06 58.42 0)
       (effects (font (size 1.27 1.27)) hide)
     )
@@
   (symbol (lib_id "power:GND") (at 179.07 96.52 0)
     (in_bom yes) (on_board yes)
-    (property "Reference" "#PWR0127" (id 0) (at 179.07 102.87 0)
+    (property "Reference" "#PWR0122" (id 0) (at 179.07 102.87 0)
       (effects (font (size 1.27 1.27)) hide)
     )
@@
   (symbol (lib_id "power:GND") (at 99.06 72.39 0)
     (in_bom yes) (on_board yes)
-    (property "Reference" "#PWR0126" (id 0) (at 99.06 78.74 0)
+    (property "Reference" "#PWR0121" (id 0) (at 99.06 78.74 0)
       (effects (font (size 1.27 1.27)) hide)
     )
@@
   (symbol (lib_id "power:+2V5") (at 193.04 90.17 0)
     (in_bom yes) (on_board yes)
-    (property "Reference" "#PWR0129" (id 0) (at 193.04 93.98 0)
+    (property "Reference" "#PWR0124" (id 0) (at 193.04 93.98 0)
       (effects (font (size 1.27 1.27)) hide)
     )
@@
   (symbol (lib_id "power:+5VP") (at 180.34 80.01 0)
     (in_bom yes) (on_board yes)
-    (property "Reference" "#PWR0128" (id 0) (at 180.34 83.82 0)
+    (property "Reference" "#PWR0123" (id 0) (at 180.34 83.82 0)
       (effects (font (size 1.27 1.27)) hide)
     )
@@
     (pin "1")
   )
+  (sheet_instances
+    (path "/" (page "1"))
+  )
+  (symbol_instances
+    (path "/00000000-0000-0000-0000-000061476b7c"
+      (reference "#PWR0120") (unit 1) (value "+10V") (footprint "")
+    )
+    (path "/00000000-0000-0000-0000-00006147a8f4"
+      (reference "#PWR0121") (unit 1) (value "GND") (footprint "")
+    )
+    (path "/00000000-0000-0000-0000-000061477276"
+      (reference "#PWR0122") (unit 1) (value "GND") (footprint "")
+    )
+    (path "/00000000-0000-0000-0000-00006171248e"
+      (reference "#PWR0123") (unit 1) (value "+5VP") (footprint "")
+    )
+    (path "/00000000-0000-0000-0000-0000616add4e"
+      (reference "#PWR0124") (unit 1) (value "+2V5") (footprint "")
+    )
+    (path "/00000000-0000-0000-0000-00006146c66c"
+      (reference "IC19") (unit 1) (value "24PCDFA6D") (footprint "SamacSys_Parts:24PCDFA6D")
+    )
+    (path "/00000000-0000-0000-0000-00006146f7fa"
+      (reference "IC20") (unit 1) (value "INA849DR") (footprint "SamacSys_Parts:SOIC127P600X175-8N")
+    )
+    (path "/00000000-0000-0000-0000-00006147457d"
+      (reference "R42") (unit 1) (value "YR1B665RCC") (footprint "SamacSys_Parts:RESAD1550W60L630D230")
+    )
+  )
 )
