File: AMS-Mega2560-Base/AMS-Mega2560-Base.kicad_pcb (KiCad board)
At the start: 4 copper layers, 168.7 x 106.7 mm, 209 parts, among them IC1 CD74HC4050ME4, IC10 LM2597MX-ADJ_NOPB, IC11 LM2597M-3.3_NOPB, IC12 OPA2340PA, IC13 MAX764CPA+, IC14 LM2917N-8_NOPB, IC15 MAX31865AAP+, IC16 DS3231SN#, IC17 MAX232CPE+, IC18 MAX31865AAP+, IC2 CD74HC4050ME4, IC3 MAX31865AAP+, IC4 MAX31865AAP+, IC5 MAX31865AAP+, IC6 LTV-814, IC7 LTV-846S, IC8 MAX31865AAP+, IC9 LM2670SX-5.0_NOPB, J1 RTD1, J10 Conn_01x03, J11 Conn_01x02, J12 Conn_01x02, J13 Conn_01x03, J14 Conn_01x02, J15 Conn_01x02, J16 Conn_01x03, J17 Conn_01x02, J18 Conn_01x02, J19 Conn_01x03, J2 RTD2, J20 Conn_01x02, J21 Screw_Terminal_01x02, J22 Conn_02x06_Odd_Even, J23 Conn_01x02, J24 Conn_01x02, J25 Conn_01x02, J26 Conn_01x03, J27 Conn_01x02, J28 Conn_01x02, J29 Conn_01x03, J3 Sense, J30 Conn_01x02, J4 Conn_02x03_Odd_Even, J5 Sense, J6 Conn_01x03, J7 Conn_01x08, J8 AdafruitUltimateGPS, J9 Conn_01x02, P1 Power, P10 CONN_01X01, P11 CONN_01X01, P12 CONN_01X01, P13 CONN_01X01, P2 Analog, P3 Analog, P4 Digital, P5 PWM, P6 PWM, P7 Communication, P8 CONN_01X01, P9 CONN_01X01, Q1 2N7000, Q10 IRF9Z34NPBF, Q11 2N7000, Q12 2N7000, Q13 IRF9Z34NPBF, Q14 IRF9Z34NPBF, Q15 2N7000, Q16 2N7000, Q17 IRF9Z34NPBF, Q18 IRF9Z34NPBF, Q19 2N7000, Q2 2N7000, Q20 IRF9Z34NPBF, Q3 2N7000, Q4 2N7000, Q5 2N7000, Q6 IRF9Z34NPBF, Q7 2N7000, Q8 2N7000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

Commit message: fixed the messed up references and cleaned up the schematic.
Parts:
- J3: value Sense -> Conn_01x08; footprint SamacSys_Parts:1727751 -> Connector_PinSocket_2.54mm:PinSocket_1x08_P2.54mm_Horizontal
- J4: value Conn_02x03_Odd_Even -> Sense1; footprint Connector_PinHeader_2.54mm:PinHeader_2x03_P2.54mm_Vertical -> SamacSys_Parts:1727751
- J5: value Sense -> Sense2
- J6: value Conn_01x03 -> AdafruitUltimateGPS; footprint Connector_PinSocket_2.54mm:PinSocket_1x03_P2.54mm_Vertical -> Connector_PinSocket_2.54mm:PinSocket_1x09_P2.54mm_Vertical
- J7: value Conn_01x08 -> Conn_02x03_Odd_Even; footprint Connector_PinSocket_2.54mm:PinSocket_1x08_P2.54mm_Horizontal -> Connector_PinHeader_2.54mm:PinHeader_2x03_P2.54mm_Vertical
- J8: value AdafruitUltimateGPS -> Conn_01x03; footprint Connector_PinSocket_2.54mm:PinSocket_1x09_P2.54mm_Vertical -> Connector_PinSocket_2.54mm:PinSocket_1x03_P2.54mm_Vertical
- moved IC15 255.7 mm to (148.6, -43.2)
- moved R36 242.9 mm to (168.3, -52.1)
- moved D9 204.1 mm to (51.0, -58.6)
- moved IC14 199.1 mm to (85.7, -54.8)
- moved J20 192.3 mm to (93.7, -7.26)
- moved J27 190.4 mm to (156.0, -42.1)
- moved R34 185.8 mm to (92.6, -45.0)
- moved R32 165.1 mm to (97.8, -52.2)
- moved IC16 163.3 mm to (60.3, -2.91)
- moved IC8 163.3 mm to (86.2, -8.30)
- moved R20 157.2 mm to (106.0, -17.3)
- moved C40 156.7 mm to (68.8, -5.66)
- moved J7 154.5 mm to (120.7, -4.47)
- moved R1 152.2 mm to (127.6, -4.77)
- moved U3 152.1 mm to (35.5, 2.01)
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Connections:
- J3 pad 1: Sense1-1 -> +5VP
- J3 pad 2: OilPressure -> unconnected-(J3-Pad2)
- J3 pad 3: Sense1-3 -> GND
- J3 pad 4: Sense1-4 -> SCLK
- J3 pad 5: FuelPressure1 -> MISO
- J3 pad 6: AFR1 -> MOSI
- J3 pad 7: Sense1-7 -> SDCS
- J3 pad 8: FuelPressure2 -> SDDetect
- J4 pad 1: unconnected-(J4-Pad1) -> Sense1-1
- J4 pad 2: unconnected-(J4-Pad2) -> OilPressure
- J4 pad 3: unconnected-(J4-Pad3) -> Sense1-3
- J4 pad 4: unconnected-(J4-Pad4) -> Sense1-4
- J4 pad 5: unconnected-(J4-Pad5) -> FuelPressure1
- J4 pad 6: unconnected-(J4-Pad6) -> AFR1
- J6 pad 1: Net-(IC2-Pad15) -> /3.3
- J6 pad 2: Net-(IC2-Pad11) -> /EN
- J6 pad 3: GND -> GPSBat
- J7 pad 2: unconnected-(J7-Pad2) -> +10V
- J7 pad 3: GND -> Vacuum1
- J7 pad 4: SCLK -> +2V5
- J7 pad 5: MISO -> Vacuum2
- J7 pad 6: MOSI -> GND
- J8 pad 1: /3.3 Logic Convert/3.3 -> Net-(IC2-Pad15)
- J8 pad 2: /3.3 Logic Convert/EN -> Net-(IC2-Pad11)
- J8 pad 3: GPSBat -> GND
Other:
- outline, holes or cut-outs redrawn
