File: AMS-Mega2560-Base/AMS-Mega2560-Base.kicad_pcb (KiCad board)
At the start: 4 copper layers, 168.7 x 106.7 mm, 209 parts, among them IC1 CD74HC4050ME4, IC10 LM2597MX-ADJ_NOPB, IC11 LM2597M-3.3_NOPB, IC12 OPA2340PA, IC13 MAX764CPA+, IC14 LM2917N-8_NOPB, IC15 MAX31865AAP+, IC16 DS3231SN#, IC17 MAX232CPE+, IC18 MAX31865AAP+, IC2 CD74HC4050ME4, IC3 MAX31865AAP+, IC4 MAX31865AAP+, IC5 MAX31865AAP+, IC6 LTV-814, IC7 LTV-846S, IC8 MAX31865AAP+, IC9 LM2670SX-5.0_NOPB, J1 RTD1, J10 Conn_01x03, J11 Conn_01x02, J12 Conn_01x02, J13 Conn_01x03, J14 Conn_01x02, J15 Conn_01x02, J16 Conn_01x03, J17 Conn_01x02, J18 Conn_01x02, J19 Conn_01x03, J2 RTD2, J20 Conn_01x02, J21 Screw_Terminal_01x02, J22 Conn_02x06_Odd_Even, J23 Conn_01x02, J24 Conn_01x02, J25 Conn_01x02, J26 Conn_01x03, J27 Conn_01x02, J28 Conn_01x02, J29 Conn_01x03, J3 Conn_01x08, J30 Conn_01x02, J4 Sense1, J5 Sense2, J6 AdafruitUltimateGPS, J7 Conn_02x03_Odd_Even, J8 Conn_01x03, J9 Conn_01x02, P1 Power, P10 CONN_01X01, P11 CONN_01X01, P12 CONN_01X01, P13 CONN_01X01, P2 Analog, P3 Analog, P4 Digital, P5 PWM, P6 PWM, P7 Communication, P8 CONN_01X01, P9 CONN_01X01, Q1 2N7000, Q10 IRF9Z34NPBF, Q11 2N7000, Q12 2N7000, Q13 IRF9Z34NPBF, Q14 IRF9Z34NPBF, Q15 2N7000, Q16 2N7000, Q17 IRF9Z34NPBF, Q18 IRF9Z34NPBF, Q19 2N7000, Q2 2N7000, Q20 IRF9Z34NPBF, Q3 2N7000, Q4 2N7000, Q5 2N7000, Q6 IRF9Z34NPBF, Q7 2N7000, Q8 2N7000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

Commit message: working on pcb layout
Parts:
- C21: value 68uF -> 0.1uF; footprint Capacitor_THT:CP_Radial_D5.0mm_P2.50mm -> Capacitor_THT:C_Rect_L9.0mm_W3.6mm_P7.50mm_MKT
- C22: value 0.1uF -> 68uF; footprint Capacitor_THT:C_Rect_L9.0mm_W3.6mm_P7.50mm_MKT -> Capacitor_THT:CP_Radial_D5.0mm_P2.50mm
- IC16, IC2: moved to B.Cu
- J22: value Conn_02x06_Odd_Even -> Conn_01x06; footprint Connector_PinSocket_2.54mm:PinSocket_2x06_P2.54mm_Vertical -> Connector_PinHeader_2.54mm:PinHeader_1x06_P2.54mm_Vertical
- moved Q6 220.9 mm to (164.5, 74.8), turned to 90 degrees
- moved U1 220.5 mm to (153.2, 79.1), turned to -90 degrees
- moved R21 208.5 mm to (159.4, 74.6), turned to 90 degrees
- moved J21 199.1 mm to (163.0, 59.7), turned to 180 degrees
- moved IC1 197.8 mm to (179.3, 131.6)
- moved D6 194.6 mm to (123.9, 50.2)
- moved J8 193.6 mm to (169.7, 128.7)
- moved IC9 190.0 mm to (133.0, 60.4), turned to 180 degrees
- moved IC2 187.0 mm to (179.3, 131.6), turned to 180 degrees
- moved U3 180.2 mm to (178.7, 111.4)
- moved L1 178.7 mm to (115.8, 49.2), turned to -90 degrees
- moved IC16 164.6 mm to (178.7, 111.4), turned to 180 degrees
- moved R22 164.0 mm to (144.3, 54.7)
- moved C15 154.6 mm to (120.7, 29.3)
- moved C16 149.5 mm to (109.6, 48.8), turned to -90 degrees
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Connections:
- C21 pad 1: +VDC -> Net-(C21-Pad1)
- C22 pad 1: Net-(C22-Pad1) -> +VDC
- IC11 pad 2: Net-(C22-Pad1) -> Net-(C21-Pad1)
- J22 pad 1: +10V -> GND
- J22 pad 2: +10V -> +2V5
- J22 pad 3: +3.3VP -> +VDC
- J22 pad 4: +3.3VP -> +5VP
- J22 pad 5: +5VP -> +3.3VP
- J22 pad 6: +5VP -> +10V
Other:
- outline, holes or cut-outs redrawn

Commit message: wip for the base PCB, finished Vacuum PCB and Fab Files for that.
Parts:
- moved J7 213.7 mm to (112.0, 106.0)
- moved J3 179.5 mm to (225.9, 109.7)
Changed lines of the file:
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@@
   )
   (footprint "Connector_PinSocket_2.54mm:PinSocket_1x08_P2.54mm_Horizontal" (layer "F.Cu")
-    (at 104.845909 -22.773913 180)
+    (at 225.93196 109.729901 180)
     (descr "Through hole angled socket strip, 1x08, 2.54mm pitch, 8.51mm socket length, single row (from Kicad 4.0.7), script generated")
     (tags "Through hole angled socket strip THT 1x08 2.54mm single row")
@@
   )
   (footprint "Connector_PinHeader_2.54mm:PinHeader_2x03_P2.54mm_Vertical" (layer "F.Cu")
-    (at 96.387378 -107.105043)
+    (at 112.042166 105.987751)
     (descr "Through hole straight pin header, 2x03, 2.54mm pitch, double rows")
     (tags "Through hole pin header THT 2x03 2.54mm double row")

Commit message: WIP for layout
Parts:
- moved R25 288.0 mm to (41.3, 127.8)
- moved R23 283.1 mm to (41.5, 120.7)
- moved D7 278.8 mm to (14.0, 114.5)
- moved L2 267.4 mm to (32.1, 100.3)
- moved IC10 266.5 mm to (44.4, 113.5)
- moved C23 262.2 mm to (6.12, 106.6)
- moved C17 258.2 mm to (27.4, 119.3)
- moved J6 254.4 mm to (254.2, 88.7)
- moved C36 249.4 mm to (161.7, 106.7), turned to 180 degrees
- moved IC17 249.3 mm to (139.3, 114.7)
- moved C19 248.3 mm to (19.7, 108.5)
- moved R38 244.2 mm to (157.2, 113.6)
- moved R37 239.7 mm to (157.2, 110.5)
- moved C13 234.3 mm to (319.4, -21.9)
- moved C14 232.8 mm to (325.3, -21.9)
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Connections:
- IC11 pad 3: unconnected-(IC11-Pad3) -> +3.3VP
- IC11 pad 4: unconnected-(IC11-Pad4) -> +3.3VP
- IC2 pad 12: Com3.3RX -> ComRX
- IC2 pad 14: Com3.3TX -> ComTX
- P7 pad 5: Com3.3TX -> /18(Tx1)
- P7 pad 6: Com3.3RX -> /19(Rx1)

Commit message: wip adding the throttle position sensor input stuff.
Parts:
- moved J21 303.6 mm to (87.0, 56.4)
- moved R21 303.6 mm to (83.4, 71.3)
- moved U1 303.6 mm to (77.1, 75.7)
- moved Q6 303.6 mm to (88.5, 71.4)
- moved C27 278.4 mm to (156.8, 175.3)
- moved C28 278.4 mm to (172.1, 180.2)
- moved C29 278.4 mm to (174.0, 171.2)
- moved C30 278.4 mm to (159.8, 189.2)
- moved C31 278.4 mm to (158.2, 197.1)
- moved C32 278.4 mm to (180.6, 190.6)
- moved C33 278.4 mm to (250.8, 177.7)
- moved C34 278.4 mm to (250.8, 171.2)
- moved C35 278.4 mm to (264.4, 171.2)
- moved D9 278.4 mm to (156.5, 170.0)
- moved IC13 278.4 mm to (172.0, 191.7)
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Other:
- outline, holes or cut-outs redrawn

Commit message: slowly working on getting the board laid out and updates to some of the schematics.
Parts:
- removed D1: 1N4007, Diode_THT:D_DO-41_SOD81_P10.16mm_Horizontal
- removed Q5: 2N7000, Package_TO_SOT_THT:TO-92_Inline
- removed R12: R, Resistor_THT:R_Axial_DIN0207_L6.3mm_D2.5mm_P2.54mm_Vertical
- added J31: Conn_01x02, Connector_PinHeader_2.54mm:PinHeader_1x02_P2.54mm_Vertical, F.Cu at (36.6, 208.6)
- added J32: Conn_01x02, Connector_PinHeader_2.54mm:PinHeader_1x02_P2.54mm_Vertical, F.Cu at (32.0, 208.6)
- added RV3: 500k, Potentiometer_THT:Potentiometer_Bourns_3296W_Vertical, F.Cu at (26.6, 216.0)
- added RV4: 500k, Potentiometer_THT:Potentiometer_Bourns_3296W_Vertical, F.Cu at (26.6, 209.5)
- C1, C10, C33, C4, C41, C8, IC5, IC8: moved to B.Cu
- C30: footprint Capacitor_THT:CP_Radial_D10.0mm_P2.50mm_P5.00mm -> Capacitor_THT:CP_Radial_D10.0mm_P5.00mm
- IC6: value LTV-814 -> OPA2340PA; footprint SamacSys_Parts:DIP762W60P254L460H450Q4N -> SamacSys_Parts:DIP794W53P254L959H508Q8N
- R27: value 4.7K -> 47k
- R28: value 4.7K -> 19.2k
- R29: value 4.7K -> 1M
- R6, R7: value R -> 47K
- moved J24 206.0 mm to (353.2, 51.4)
- moved RV2 206.0 mm to (364.2, 40.6)
- moved C27 206.0 mm to (316.1, 44.8)
- moved C28 206.0 mm to (331.4, 49.7)
- moved C29 206.0 mm to (333.4, 40.7)
- moved C32 206.0 mm to (340.0, 60.1)
- moved IC13 206.0 mm to (331.3, 61.2)
- moved IC14 206.0 mm to (350.6, 43.3)
- moved J23 206.0 mm to (358.4, 46.2)
- moved R33 206.0 mm to (338.5, 66.6)
- moved R34 206.0 mm to (357.5, 53.1)
- moved RV1 206.0 mm to (347.8, 52.3)
- moved C31 206.0 mm to (317.6, 66.7)
- moved D9 206.0 mm to (315.9, 39.5)
- moved L4 206.0 mm to (315.9, 50.5)
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Connections:
- IC6 pad 1: Net-(IC6-Pad1) -> ThrottlePositionADC
- IC6 pad 2: Net-(D1-Pad2) -> ThrottlePositionADC
- IC6 pad 3: GND -> Net-(IC6-Pad3)
- IC6 pad 4: Logging -> GND
- IC7 pad 10: IN4 -> Logging
- P3 pad 5: /A12 -> ThrottlePositionADC
- P3 pad 6: /A13 -> SpareBufferedADC
- P4 pad 10: IN4 -> IN3
- P4 pad 12: IN3 -> OUTPUTLED2
- P4 pad 14: OUTPUTLED2 -> OUTPUTLED1
- P4 pad 16: OUTPUTLED1 -> /41
- Q1 pad 3: Net-(D1-Pad1) -> Net-(D5-Pad1)
- R19 pad 2: IN4 -> Logging
- R6 pad 1: +5VP -> GND
- R6 pad 2: Net-(IC6-Pad1) -> ThrottlePositionADC
- R7 pad 1: +5VP -> GND
- R7 pad 2: Logging -> SpareBufferedADC
Other:
- board text added: "10V"
- board text added: "2"
- board text added: "2-3"
- board text added: "2-4"
- board text added: "2.5V"
- board text added: "3"
- board text added: "3.3V"
- board text added: "5V"
- board text added: "GND"
- board text added: "VDC"

Commit message: wip
Parts:
- moved IC12 154.2 mm to (137.4, 131.9)
- moved R30 149.8 mm to (141.2, 139.0), turned to 180 degrees
- moved R27 149.2 mm to (130.7, 131.2), turned to -90 degrees
- moved R29 145.5 mm to (136.0, 139.0), turned to 180 degrees
- moved R28 145.2 mm to (130.7, 136.4), turned to -90 degrees
- moved RV3 138.0 mm to (129.3, 123.7)
- moved RV4 137.4 mm to (129.3, 118.2)
- moved IC6 136.2 mm to (137.3, 121.0)
- moved R7 130.1 mm to (144.0, 124.8), turned to 90 degrees
- moved J32 127.2 mm to (119.8, 116.6)
- moved R31 122.6 mm to (118.5, 110.3)
- moved J31 119.5 mm to (119.8, 122.9)
- moved R6 117.5 mm to (147.1, 124.8), turned to 90 degrees
- moved U2 110.9 mm to (120.1, 107.3), turned to 90 degrees
- moved C21 94.7 mm to (124.9, 51.0), turned to 180 degrees
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Routing:
- net +VDC: track 0.00 -> 335.9 mm
- net GND: track 0.00 -> 79.0 mm
- net +10V: track 0.00 -> 64.2 mm
- net Sense2-3: track 0.00 -> 54.4 mm, vias 0 -> 1
- net Net-(Q18-Pad1): track 0.00 -> 50.4 mm
- net Sense1-7: track 0.00 -> 48.1 mm
- net Sense1-4: track 0.00 -> 42.1 mm
- net Sense1-1: track 0.00 -> 34.9 mm
- net Sense2-6: track 0.00 -> 34.4 mm
- net Net-(C21-Pad1): track 0.00 -> 27.2 mm
- net Sense2-9: track 0.00 -> 26.9 mm
- net +3.3VP: track 0.00 -> 25.4 mm
- net Net-(Q14-Pad1): track 0.00 -> 24.7 mm
- net Net-(C15-Pad1): track 0.00 -> 21.1 mm
- net +5VP: track 0.00 -> 20.8 mm
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- added copper zone on B.Cu, net GND
- added copper zone on F.Cu, net GND
Other:
- board text added: "+V"

Commit message: WIP for layout.
Parts:
- C1, C10, C11, C2, C33, C34, C4, C41, C42, C5, C7, C8: footprint Capacitor_THT:C_Disc_D7.5mm_W5.0mm_P10.00mm -> Capacitor_SMD:C_0805_2012Metric_Pad1.18x1.45mm_HandSolder
- C31, IC15, Z2, Z4, Z6: moved to B.Cu
- moved C2 232.6 mm to (353.7, 154.9)
- moved C3 232.6 mm to (367.2, 154.9)
- moved J11 232.6 mm to (364.5, 170.2)
- moved J9 232.6 mm to (372.4, 160.5)
- moved R1 232.6 mm to (365.7, 180.6)
- moved C1 232.6 mm to (357.6, 158.6)
- moved IC3 232.6 mm to (357.0, 169.1)
- moved J10 232.6 mm to (367.8, 160.5)
- moved R2 232.6 mm to (376.8, 160.2)
- moved J23 188.6 mm to (175.8, 93.4)
- moved C7 165.3 mm to (376.0, 107.6)
- moved C8 165.3 mm to (382.2, 113.5)
- moved C9 165.3 mm to (385.4, 113.9)
- moved J15 165.3 mm to (390.6, 119.5)
- moved J17 165.3 mm to (382.7, 129.2)
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Routing:
- net Net-(IC9-Pad5): track 3.73 -> 18.9 mm
- net GND: track 79.0 -> 68.9 mm
- net +5VP: track 20.8 -> 28.1 mm
- net Net-(C15-Pad2): track 17.8 -> 19.9 mm
- net Net-(C15-Pad1): track 21.1 -> 23.2 mm
- net +VDC: track 335.9 -> 337.8 mm
Other:
- outline, holes or cut-outs redrawn

Commit message: continuing pcb layout
Parts:
- C1, C33, C4, C8, IC15, IC5, IC8: moved to F.Cu
- C11, C42: moved to B.Cu
- moved IC15 182.5 mm to (344.9, 33.7), turned to 0 degrees
- moved C33 177.5 mm to (352.5, 26.8)
- moved C34 177.5 mm to (348.5, 23.0)
- moved C35 177.5 mm to (362.1, 23.0)
- moved J25 177.5 mm to (367.3, 28.6)
- moved J26 177.5 mm to (362.6, 28.6)
- moved J27 177.5 mm to (359.3, 38.3)
- moved R36 177.5 mm to (371.6, 28.3)
- moved R5 140.8 mm to (104.9, 127.5), turned to -90 degrees
- moved J28 136.8 mm to (194.9, 117.9)
- moved J30 136.8 mm to (191.2, 117.9)
- moved J29 136.1 mm to (198.5, 117.8)
- moved R10 135.2 mm to (105.4, 134.2), turned to -90 degrees
- moved Q1 134.7 mm to (101.8, 128.4), turned to 180 degrees
- moved R9 130.1 mm to (105.2, 140.7), turned to -90 degrees
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Routing:
- net GND: track 68.9 -> 73.6 mm
- net Net-(Q6-Pad1): track 5.17 -> 7.29 mm
Other:
- board text added: "Left Side Temp"
- board text added: "WaterTemp"
