File: AMS-Mega2560-Base/file614CA8F2.kicad_sch (KiCad schematic)
At the start: 18 parts, among them IC11 MAX764CPA+, IC12 LM2917N-8_NOPB, J22 Conn_01x02, J23 Conn_01x02

Commit message: fixing some library settings and updating some schematics
Parts:
- R25, R26, R27, R28: footprint Resistor_THT:R_Axial_DIN0207_L6.3mm_D2.5mm_P5.08mm_Vertical -> Resistor_THT:R_Axial_DIN0207_L6.3mm_D2.5mm_P2.54mm_Vertical
Changed lines of the file:
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@@
       (effects (font (size 1.27 1.27)) (justify left))
     )
-    (property "Footprint" "Resistor_THT:R_Axial_DIN0207_L6.3mm_D2.5mm_P5.08mm_Vertical" (id 2) (at 150.622 87.63 90)
+    (property "Footprint" "Resistor_THT:R_Axial_DIN0207_L6.3mm_D2.5mm_P2.54mm_Vertical" (id 2) (at 150.622 87.63 90)
       (effects (font (size 1.27 1.27)) hide)
     )
@@
       (effects (font (size 1.27 1.27)) (justify left))
     )
-    (property "Footprint" "Resistor_THT:R_Axial_DIN0207_L6.3mm_D2.5mm_P5.08mm_Vertical" (id 2) (at 150.622 100.33 90)
+    (property "Footprint" "Resistor_THT:R_Axial_DIN0207_L6.3mm_D2.5mm_P2.54mm_Vertical" (id 2) (at 150.622 100.33 90)
       (effects (font (size 1.27 1.27)) hide)
     )
@@
     (property "Reference" "R28" (id 0) (at 243.84 93.8022 90))
     (property "Value" "470" (id 1) (at 243.84 96.1136 90))
-    (property "Footprint" "Resistor_THT:R_Axial_DIN0207_L6.3mm_D2.5mm_P5.08mm_Vertical" (id 2) (at 243.84 100.838 90)
+    (property "Footprint" "Resistor_THT:R_Axial_DIN0207_L6.3mm_D2.5mm_P2.54mm_Vertical" (id 2) (at 243.84 100.838 90)
       (effects (font (size 1.27 1.27)) hide)
     )
@@
       (effects (font (size 1.27 1.27)) (justify left))
     )
-    (property "Footprint" "Resistor_THT:R_Axial_DIN0207_L6.3mm_D2.5mm_P5.08mm_Vertical" (id 2) (at 174.752 125.73 90)
+    (property "Footprint" "Resistor_THT:R_Axial_DIN0207_L6.3mm_D2.5mm_P2.54mm_Vertical" (id 2) (at 174.752 125.73 90)
       (effects (font (size 1.27 1.27)) hide)
     )

Commit message: BaseBoard fixes and updates. doing schematic work.
Parts:
- C28: footprint Capacitor_THT:CP_Radial_D10.0mm_P2.50mm_P5.00mm -> Capacitor_THT:CP_Radial_D10.0mm_P5.00mm
- renumbered D4 to D9, IC11 to IC13, IC12 to IC14, J22 to J23, J23 to J24, R25 to R32, R26 to R33, R27 to R34, R28 to R35
Changed lines of the file:
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@@
   (symbol (lib_id "SamacSys_Parts:MAX764CPA+") (at 40.64 48.26 0) (unit 1)
     (in_bom yes) (on_board yes)
-    (property "Reference" "IC11" (id 0) (at 54.61 41.529 0))
+    (property "Reference" "IC13" (id 0) (at 54.61 41.529 0))
     (property "Value" "MAX764CPA+" (id 1) (at 54.61 43.8404 0))
     (property "Footprint" "SamacSys_Parts:DIP762W56P254L938H457Q8N" (id 2) (at 64.77 45.72 0)
@@
   (symbol (lib_id "SamacSys_Parts:LM2917N-8_NOPB") (at 186.69 93.98 0) (unit 1)
     (in_bom yes) (on_board yes)
-    (property "Reference" "IC12" (id 0) (at 205.74 87.249 0))
+    (property "Reference" "IC14" (id 0) (at 205.74 87.249 0))
     (property "Value" "LM2917N-8_NOPB" (id 1) (at 205.74 89.5604 0))
     (property "Footprint" "SamacSys_Parts:DIP794W53P254L959H508Q8N" (id 2) (at 220.98 91.44 0)
@@
   (symbol (lib_id "power:GND") (at 20.32 69.85 0) (unit 1)
     (in_bom yes) (on_board yes)
-    (property "Reference" "#PWR081" (id 0) (at 20.32 76.2 0)
+    (property "Reference" "#PWR083" (id 0) (at 20.32 76.2 0)
       (effects (font (size 1.27 1.27)) hide)
     )
@@
   (symbol (lib_id "power:+10V") (at 92.71 50.8 0) (unit 1)
     (in_bom yes) (on_board yes)
-    (property "Reference" "#PWR082" (id 0) (at 92.71 54.61 0)
+    (property "Reference" "#PWR084" (id 0) (at 92.71 54.61 0)
       (effects (font (size 1.27 1.27)) hide)
     )
@@
   (symbol (lib_id "power:+VDC") (at 251.46 93.98 0) (unit 1)
     (in_bom yes) (on_board yes)
-    (property "Reference" "#PWR086" (id 0) (at 251.46 96.52 0)
+    (property "Reference" "#PWR088" (id 0) (at 251.46 96.52 0)
       (effects (font (size 1.27 1.27)) hide)
     )
@@
       (effects (font (size 1.27 1.27)) (justify left))
     )
-    (property "Footprint" "Capacitor_THT:CP_Radial_D10.0mm_P2.50mm_P5.00mm" (id 2) (at 80.01 62.23 0)
+    (property "Footprint" "Capacitor_THT:CP_Radial_D10.0mm_P5.00mm" (id 2) (at 80.01 62.23 0)
       (effects (font (size 1.27 1.27)) hide)
     )
@@
   (symbol (lib_id "SamacSys_Parts:1N5817") (at 101.6 44.45 0) (unit 1)
     (in_bom yes) (on_board yes)
-    (property "Reference" "D4" (id 0) (at 109.22 37.6682 0))
+    (property "Reference" "D9" (id 0) (at 109.22 37.6682 0))
     (property "Value" "1N5817" (id 1) (at 109.22 39.9796 0))
     (property "Footprint" "SamacSys_Parts:DIOAD1414W86L464D238" (id 2) (at 113.03 44.45 0)
@@
   (symbol (lib_id "Connector_Generic:Conn_01x02") (at 148.59 62.23 0) (unit 1)
     (in_bom yes) (on_board yes)
-    (property "Reference" "J23" (id 0) (at 150.622 62.4332 0)
+    (property "Reference" "J24" (id 0) (at 150.622 62.4332 0)
       (effects (font (size 1.27 1.27)) (justify left))
     )
@@
   (symbol (lib_id "Device:R") (at 152.4 87.63 0) (unit 1)
     (in_bom yes) (on_board yes)
-    (property "Reference" "R25" (id 0) (at 154.178 86.4616 0)
+    (property "Reference" "R32" (id 0) (at 154.178 86.4616 0)
       (effects (font (size 1.27 1.27)) (justify left))
     )
@@
   (symbol (lib_id "Device:R") (at 152.4 100.33 0) (unit 1)
     (in_bom yes) (on_board yes)
-    (property "Reference" "R26" (id 0) (at 154.178 99.1616 0)
+    (property "Reference" "R33" (id 0) (at 154.178 99.1616 0)
       (effects (font (size 1.27 1.27)) (justify left))
     )
@@
   (symbol (lib_id "power:GND") (at 152.4 110.49 0) (unit 1)
     (in_bom yes) (on_board yes)
-    (property "Reference" "#PWR083" (id 0) (at 152.4 116.84 0)
+    (property "Reference" "#PWR085" (id 0) (at 152.4 116.84 0)
       (effects (font (size 1.27 1.27)) hide)
     )
@@
   (symbol (lib_id "power:GND") (at 237.49 93.98 0) (unit 1)
     (in_bom yes) (on_board yes)
-    (property "Reference" "#PWR085" (id 0) (at 237.49 100.33 0)
+    (property "Reference" "#PWR087" (id 0) (at 237.49 100.33 0)
       (effects (font (size 1.27 1.27)) hide)
     )
@@
   (symbol (lib_id "power:GND") (at 186.69 134.62 0) (unit 1)
     (in_bom yes) (on_board yes)
-    (property "Reference" "#PWR084" (id 0) (at 186.69 140.97 0)
+    (property "Reference" "#PWR086" (id 0) (at 186.69 140.97 0)
       (effects (font (size 1.27 1.27)) hide)
     )
@@
   (symbol (lib_id "Device:R") (at 243.84 99.06 90) (unit 1)
     (in_bom yes) (on_board yes)
-    (property "Reference" "R28" (id 0) (at 243.84 93.8022 90))
+    (property "Reference" "R35" (id 0) (at 243.84 93.8022 90))
     (property "Value" "470" (id 1) (at 243.84 96.1136 90))
     (property "Footprint" "Resistor_THT:R_Axial_DIN0207_L6.3mm_D2.5mm_P2.54mm_Vertical" (id 2) (at 243.84 100.838 90)
@@
   (symbol (lib_id "Device:R") (at 176.53 125.73 0) (unit 1)
     (in_bom yes) (on_board yes)
-    (property "Reference" "R27" (id 0) (at 178.308 124.5616 0)
+    (property "Reference" "R34" (id 0) (at 178.308 124.5616 0)
       (effects (font (size 1.27 1.27)) (justify left))
     )
@@
   (symbol (lib_id "Connector_Generic:Conn_01x02") (at 97.79 50.8 0) (unit 1)
     (in_bom yes) (on_board yes)
-    (property "Reference" "J22" (id 0) (at 99.822 51.0032 0)
-      (effects (font (size 1.27 1.27)) (justify left))
-    )
+    (property "Reference" "J23" (id 0) (at 99.822 51.0032 0)
+      (effects (font (size 1.27 1.27)) (justify left))
+    )

Commit message: slowly working on getting the board laid out and updates to some of the schematics.
Parts:
- C30: footprint Capacitor_THT:CP_Radial_D10.0mm_P2.50mm_P5.00mm -> Capacitor_THT:CP_Radial_D10.0mm_P5.00mm
Changed lines of the file:
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@@
       (effects (font (size 1.27 1.27)) (justify left))
     )
-    (property "Footprint" "Capacitor_THT:CP_Radial_D10.0mm_P2.50mm_P5.00mm" (id 2) (at 116.84 62.23 0)
+    (property "Footprint" "Capacitor_THT:CP_Radial_D10.0mm_P5.00mm" (id 2) (at 116.84 62.23 0)
       (effects (font (size 1.27 1.27)) hide)
     )
