File: AMS-Mega2560-Base/AMS-Mega2560-Base.kicad_sch (KiCad schematic)
At the start: 28 parts, among them J1 Conn_01x03, J2 Conn_01x03, J3 Conn_01x08, J4 Sense1, J5 Sense2, J6 AdafruitUltimateGPS, J7 Conn_02x03_Odd_Even, J8 Conn_01x03, P1 Power, P10 CONN_01X01, P11 CONN_01X01, P12 CONN_01X01, P13 CONN_01X01, P2 Analog, P3 Analog, P4 Digital, P5 PWM, P6 PWM, P7 Communication, P8 CONN_01X01, P9 CONN_01X01, T1 Conn_01x08, T2 Conn_01x08, T3 Conn_01x08, T4 Conn_01x08, T5 Conn_01x08, T6 Conn_01x08

Commit message: wip while i get set to autoroute
Parts:
- added J9: Conn_01x03, Connector_PinHeader_2.54mm:PinHeader_1x03_P2.54mm_Vertical, symbol Connector_Generic:Conn_01x03
Connections:
- net GND: now also J9.3 (Pin_3)
- net Sheet6152913C/RSCOM2RX: now also J9.2 (Pin_2)
- net Sheet6152913C/RSCOM2TX: now also J9.1 (Pin_1)
Changed lines of the file:
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@@
     (stroke (width 0) (type default) (color 0 0 0 0))
   )
+  (wire (pts (xy 269.24 73.025) (xy 276.86 73.025))
+    (stroke (width 0) (type default) (color 0 0 0 0))
+  )
   (wire (pts (xy 355.6 49.53) (xy 353.06 49.53))
     (stroke (width 0) (type default) (color 0 0 0 0))
   )
+  (wire (pts (xy 269.24 78.105) (xy 269.24 80.645))
+    (stroke (width 0) (type default) (color 0 0 0 0))
+  )
   (wire (pts (xy 344.17 142.24) (xy 337.82 142.24))
     (stroke (width 0) (type default) (color 0 0 0 0))
@@
     (stroke (width 0) (type default) (color 0 0 0 0))
   )
+  (wire (pts (xy 269.24 75.565) (xy 276.86 75.565))
+    (stroke (width 0) (type default) (color 0 0 0 0))
+  )
   (wire (pts (xy 194.31 35.56) (xy 198.12 35.56))
     (stroke (width 0) (type default) (color 0 0 0 0))
@@
     (pin "1")
   )
+  (symbol (lib_id "Connector_Generic:Conn_01x03") (at 264.16 75.565 0) (mirror y) (unit 1)
+    (in_bom yes) (on_board yes) (fields_autoplaced)
+    (property "Reference" "J9" (id 0) (at 264.16 67.7885 0))
+    (property "Value" "Conn_01x03" (id 1) (at 264.16 70.5636 0))
+    (property "Footprint" "Connector_PinHeader_2.54mm:PinHeader_1x03_P2.54mm_Vertical" (id 2) (at 264.16 75.565 0)
+      (effects (font (size 1.27 1.27)) hide)
+    )
+    (property "Datasheet" "~" (id 3) (at 264.16 75.565 0)
+      (effects (font (size 1.27 1.27)) hide)
+    )
+    (pin "1")
+    (pin "2")
+    (pin "3")
+  )
   (symbol (lib_id "power:+5V") (at 69.215 240.03 270) (unit 1)
     (in_bom yes) (on_board yes) (fields_autoplaced)
@@
     (pin "9")
   )
+  (symbol (lib_id "power:GND") (at 269.24 80.645 0) (unit 1)
+    (in_bom yes) (on_board yes)
+    (property "Reference" "#PWR049" (id 0) (at 269.24 86.995 0)
+      (effects (font (size 1.27 1.27)) hide)
+    )
+    (property "Value" "GND" (id 1) (at 269.24 84.455 0))
+    (property "Footprint" "" (id 2) (at 269.24 80.645 0))
+    (property "Datasheet" "" (id 3) (at 269.24 80.645 0))
+    (pin "1")
+  )
   (symbol (lib_id "Connector_Generic:Conn_01x08") (at 56.515 247.65 0) (mirror y) (unit 1)
     (in_bom yes) (on_board yes)
@@
       (effects (font (size 1.27 1.27)) (justify right))
     )
-    (pin "RSCOM2TX" input (at 276.86 73.66 180)
+    (pin "RSCOM2TX" input (at 276.86 73.025 180)
       (effects (font (size 1.27 1.27)) (justify left))
     )
@@
       (reference "#PWR048") (unit 1) (value "GND") (footprint "")
     )
+    (path "/8bc4232b-d531-4586-83da-9fe48c419417"
+      (reference "#PWR049") (unit 1) (value "GND") (footprint "")
+    )
     (path "/00000000-0000-0000-0000-000061493c0e/00000000-0000-0000-0000-0000614baf40"
       (reference "#PWR053") (unit 1) (value "GND") (footprint "")
@@
       (reference "J8") (unit 1) (value "Conn_01x03") (footprint "Connector_PinHeader_2.54mm:PinHeader_1x03_P2.54mm_Vertical")
     )
+    (path "/3fd9261e-2ed9-4c7f-b607-da78646bf5d3"
+      (reference "J9") (unit 1) (value "Conn_01x03") (footprint "Connector_PinHeader_2.54mm:PinHeader_1x03_P2.54mm_Vertical")
+    )
     (path "/00000000-0000-0000-0000-000061493c0e/f43ecda4-cf8e-4f4b-970d-8c733cfa2ce0"
