File: AMS-Mega2560-Base/BufferedADC.kicad_sch (KiCad schematic)
At the start: 9 parts, among them IC20 OPA4340UA

Commit message: working on this.
Parts:
- IC6: renamed from IC20; footprint SOIC127P600X175-14N -> SamacSys_Parts:SOIC127P600X175-14N
- renumbered R36 to R2, R72 to R20, R60 to R3, R71 to R4, R64 to R6, R66 to R68, R67 to R69, R65 to R7
Other:
- moved on the sheet: IC6, R2, R20, R3, R4, R6, R68, R69, R7
