File: AMS-Vacuum-Sensor/AMS-Vacuum-Sensor.kicad_sch (KiCad schematic)
At the start: 7 parts, among them IC1 24PCDFA6D, IC2 24PCDFA6D, IC3 INA849DR, IC4 INA849DR, J1 Conn_02x03_Odd_Even

Commit message: wip for the base PCB, finished Vacuum PCB and Fab Files for that.
Changed lines of the file:
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@@
 (kicad_sch (version 20211123) (generator eeschema)
   (paper "A4")
+  (junction (at 254 110.49) (diameter 0) (color 0 0 0 0)
+  )
+  (junction (at 256.54 95.25) (diameter 0) (color 0 0 0 0)
+  )
+  (junction (at 264.16 92.71) (diameter 0) (color 0 0 0 0)
+  )
+  (junction (at 234.95 93.98) (diameter 0) (color 0 0 0 0)
+  )
+  (wire (pts (xy 264.16 92.71) (xy 271.78 92.71))
+    (stroke (width 0) (type default) (color 0 0 0 0))
+  )
   (wire (pts (xy 102.87 125.73) (xy 100.33 125.73))
     (stroke (width 0) (type default) (color 0 0 0 0))
@@
     (stroke (width 0) (type default) (color 0 0 0 0))
   )
-  (wire (pts (xy 256.54 92.71) (xy 256.54 100.33))
+  (wire (pts (xy 256.54 92.71) (xy 256.54 95.25))
     (stroke (width 0) (type default) (color 0 0 0 0))
   )
@@
     (stroke (width 0) (type default) (color 0 0 0 0))
   )
+  (wire (pts (xy 256.54 95.25) (xy 256.54 100.33))
+    (stroke (width 0) (type default) (color 0 0 0 0))
+  )
   (wire (pts (xy 100.33 123.19) (xy 137.16 123.19))
     (stroke (width 0) (type default) (color 0 0 0 0))
@@
     (stroke (width 0) (type default) (color 0 0 0 0))
   )
+  (wire (pts (xy 254 110.49) (xy 260.35 110.49))
+    (stroke (width 0) (type default) (color 0 0 0 0))
+  )
   (wire (pts (xy 190.5 105.41) (xy 238.76 105.41))
     (stroke (width 0) (type default) (color 0 0 0 0))
@@
     (stroke (width 0) (type default) (color 0 0 0 0))
   )
-  (wire (pts (xy 234.95 92.71) (xy 234.95 100.33))
+  (wire (pts (xy 251.46 95.25) (xy 256.54 95.25))
+    (stroke (width 0) (type default) (color 0 0 0 0))
+  )
+  (wire (pts (xy 234.95 92.71) (xy 234.95 93.98))
     (stroke (width 0) (type default) (color 0 0 0 0))
   )
@@
     (stroke (width 0) (type default) (color 0 0 0 0))
   )
+  (wire (pts (xy 226.06 93.98) (xy 234.95 93.98))
+    (stroke (width 0) (type default) (color 0 0 0 0))
+  )
   (wire (pts (xy 180.34 85.09) (xy 180.34 80.01))
     (stroke (width 0) (type default) (color 0 0 0 0))
   )
+  (wire (pts (xy 234.95 93.98) (xy 234.95 100.33))
+    (stroke (width 0) (type default) (color 0 0 0 0))
+  )
   (wire (pts (xy 110.49 144.78) (xy 110.49 128.27))
     (stroke (width 0) (type default) (color 0 0 0 0))
@@
   )
   (wire (pts (xy 96.52 63.5) (xy 133.35 63.5))
+    (stroke (width 0) (type default) (color 0 0 0 0))
+  )
+  (wire (pts (xy 251.46 90.17) (xy 251.46 95.25))
     (stroke (width 0) (type default) (color 0 0 0 0))
   )
@@
     (pin "1")
   )
+  (symbol (lib_id "power:PWR_FLAG") (at 251.46 90.17 0) (unit 1)
+    (in_bom yes) (on_board yes) (fields_autoplaced)
+    (property "Reference" "#FLG0103" (id 0) (at 251.46 88.265 0)
+      (effects (font (size 1.27 1.27)) hide)
+    )
+    (property "Value" "PWR_FLAG" (id 1) (at 251.46 86.5655 0))
+    (property "Footprint" "" (id 2) (at 251.46 90.17 0)
+      (effects (font (size 1.27 1.27)) hide)
+    )
+    (property "Datasheet" "~" (id 3) (at 251.46 90.17 0)
+      (effects (font (size 1.27 1.27)) hide)
+    )
+    (pin "1")
+  )
   (symbol (lib_id "power:+5VP") (at 184.15 139.7 0) (unit 1)
     (in_bom yes) (on_board yes)
@@
     (pin "1")
   )
+  (symbol (lib_id "power:PWR_FLAG") (at 271.78 92.71 0) (unit 1)
+    (in_bom yes) (on_board yes) (fields_autoplaced)
+    (property "Reference" "#FLG0101" (id 0) (at 271.78 90.805 0)
+      (effects (font (size 1.27 1.27)) hide)
+    )
+    (property "Value" "PWR_FLAG" (id 1) (at 271.78 89.1055 0))
+    (property "Footprint" "" (id 2) (at 271.78 92.71 0)
+      (effects (font (size 1.27 1.27)) hide)
+    )
+    (property "Datasheet" "~" (id 3) (at 271.78 92.71 0)
+      (effects (font (size 1.27 1.27)) hide)
+    )
+    (pin "1")
+  )
   (symbol (lib_id "power:+2V5") (at 264.16 92.71 0) (unit 1)
     (in_bom yes) (on_board yes)
@@
     )
     (property "Datasheet" "" (id 3) (at 234.95 92.71 0)
+      (effects (font (size 1.27 1.27)) hide)
+    )
+    (pin "1")
+  )
+  (symbol (lib_id "power:GNDPWR") (at 260.35 110.49 0) (unit 1)
+    (in_bom yes) (on_board yes) (fields_autoplaced)
+    (property "Reference" "#PWR?" (id 0) (at 260.35 115.57 0)
+      (effects (font (size 1.27 1.27)) hide)
+    )
+    (property "Value" "GNDPWR" (id 1) (at 260.223 114.6461 0))
+    (property "Footprint" "" (id 2) (at 260.35 111.76 0)
+      (effects (font (size 1.27 1.27)) hide)
+    )
+    (property "Datasheet" "" (id 3) (at 260.35 111.76 0)
       (effects (font (size 1.27 1.27)) hide)
     )
@@
     (pin "8")
   )
+  (symbol (lib_id "power:PWR_FLAG") (at 226.06 93.98 0) (unit 1)
+    (in_bom yes) (on_board yes) (fields_autoplaced)
+    (property "Reference" "#FLG0102" (id 0) (at 226.06 92.075 0)
+      (effects (font (size 1.27 1.27)) hide)
+    )
+    (property "Value" "PWR_FLAG" (id 1) (at 226.06 90.3755 0))
+    (property "Footprint" "" (id 2) (at 226.06 93.98 0)
+      (effects (font (size 1.27 1.27)) hide)
+    )
+    (property "Datasheet" "~" (id 3) (at 226.06 93.98 0)
+      (effects (font (size 1.27 1.27)) hide)
+    )
+    (pin "1")
+  )
   (symbol (lib_id "power:GND") (at 254 110.49 0) (unit 1)
     (in_bom yes) (on_board yes)
@@
   )
   (symbol_instances
+    (path "/9841377f-19fe-4848-82b2-954ed8fd28f4"
+      (reference "#FLG0101") (unit 1) (value "PWR_FLAG") (footprint "")
+    )
+    (path "/d873b872-9a03-4cc9-b5be-869bca30656a"
+      (reference "#FLG0102") (unit 1) (value "PWR_FLAG") (footprint "")
+    )
+    (path "/083b2527-e405-49bd-a309-2cdb85cd9a7a"
+      (reference "#FLG0103") (unit 1) (value "PWR_FLAG") (footprint "")
+    )
     (path "/00000000-0000-0000-0000-000061476b7c"
       (reference "#PWR01") (unit 1) (value "+10V") (footprint "")
@@
       (reference "#PWR014") (unit 1) (value "+2V5") (footprint "")
     )
+    (path "/a5419243-521f-4e0e-87a5-68bb7d8c3242"
+      (reference "#PWR?") (unit 1) (value "GNDPWR") (footprint "")
+    )
     (path "/00000000-0000-0000-0000-00006146c66c"
