File: AMS-Vacuum-Sensor/AMS-Vacuum-Sensor.kicad_pcb (KiCad board)
At the start: 2 copper layers, 7 parts, among them IC1 24PCDFA6D, IC2 24PCDFA6D, IC3 INA849DR, IC4 INA849DR, J1 Conn_02x03_Odd_Even

Commit message: wip for the base PCB, finished Vacuum PCB and Fab Files for that.
Parts:
- IC3, IC4, R1, R2: moved to B.Cu
- moved IC3 63.5 mm to (110.1, 100.5), turned to -90 degrees
- moved J1 59.8 mm to (115.6, 110.0)
- moved R2 35.5 mm to (131.4, 87.3), turned to -90 degrees
- moved R1 32.3 mm to (103.5, 87.3), turned to -90 degrees
- moved IC4 31.7 mm to (125.0, 100.5), turned to -90 degrees
- moved IC2 14.5 mm to (128.7, 91.9)
- moved IC1 13.6 mm to (113.8, 91.9)
Routing:
- net GND: track 0.00 -> 61.8 mm, vias 0 -> 1
- net +10V: track 0.00 -> 44.6 mm, vias 0 -> 1
- net +2V5: track 0.00 -> 33.1 mm
- net +5VP: track 0.00 -> 30.2 mm, vias 0 -> 2
- net Net-(IC4-Pad7): track 0.00 -> 24.9 mm, vias 0 -> 1
- net Net-(IC4-Pad2): track 0.00 -> 15.3 mm
- net Net-(IC3-Pad7): track 0.00 -> 13.4 mm
- net Net-(IC3-Pad2): track 0.00 -> 13.0 mm
- net Net-(IC3-Pad3): track 0.00 -> 10.6 mm
- net Net-(IC4-Pad3): track 0.00 -> 8.45 mm
- net Net-(IC1-Pad4): track 0.00 -> 7.66 mm, vias 0 -> 1
- net Net-(IC2-Pad4): track 0.00 -> 6.63 mm
- net Net-(IC2-Pad2): track 0.00 -> 6.13 mm
- net Net-(IC1-Pad2): track 0.00 -> 6.13 mm
Other:
- board outline added: 31.8 x 41.3 mm
- board text added: "Vac1"
- board text added: "Vac2"
- board text added: "Vers. 1.0"
