File: AMS-Mega2560-Base-Lack-Of-Chips/AMS-Mega2560-Base-Lack-Of-Chips.kicad_pcb (KiCad board)
At the start: 4 copper layers, 168.7 x 106.7 mm, 231 parts, among them IC1 CD74HC4050ME4, IC10 LM2597MX-ADJ_NOPB, IC11 LM2597M-3.3_NOPB, IC12 OPA2340PA, IC13 MAX764CPA+, IC14 LM2917N-8_NOPB, IC15 MAX31865AAP+, IC16 DS3231SN#, IC17 MAX232CPE+, IC18 MAX31865AAP+, IC19 MAX6326UR31+T, IC2 CD74HC4050ME4, IC20 OPA4340UA, IC3 MAX31865AAP+, IC4 MAX31865AAP+, IC5 MAX31865AAP+, IC6 OPA4340UA, IC7 LTV-846S, IC8 MAX31865AAP+, IC9 LM2670SX-5.0_NOPB, J1 RTD1, J10 Conn_01x03, J11 Conn_01x02, J12 Conn_01x02, J13 Conn_01x03, J14 Conn_01x02, J15 Conn_01x02, J16 Conn_01x03, J17 Conn_01x02, J18 Conn_01x02, J19 Conn_01x03, J2 RTD2, J20 Conn_01x02, J21 Screw_Terminal_01x03, J22 Conn_01x07, J23 Conn_01x02, J24 Conn_01x02, J25 Conn_01x02, J26 Conn_01x03, J27 Conn_01x02, J28 Conn_01x02, J29 Conn_01x03, J3 Conn_01x08, J30 Conn_01x02, J31 Conn_01x02, J4 Sense1, J5 Sense2, J6 AdafruitUltimateGPS, J7 Conn_02x03_Odd_Even, J8 Conn_01x03, J9 Conn_01x02, K1 DIP05-1A72-12L, P1 Power, P10 CONN_01X01, P11 CONN_01X01, P12 CONN_01X01, P13 CONN_01X01, P2 Analog, P3 Analog, P4 Digital, P5 PWM, P6 PWM, P7 Communication, P8 CONN_01X01, P9 CONN_01X01, Q1 2N7000, Q10 IRF9Z34NPBF, Q11 2N7000, Q12 2N7000, Q13 IRF9Z34NPBF, Q14 IRF9Z34NPBF, Q15 2N7000, Q16 2N7000, Q17 IRF9Z34NPBF, Q18 IRF9Z34NPBF, Q19 2N7000, Q2 2N7000, Q20 IRF9Z34NPBF, Q21 IRF9Z34NPBF, Q22 IRF9610PBF-BE3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

Commit message: updating some Resistor values
Parts:
- removed C1, C10, C11, C2, C33, C34, C4, C41, C42, C5, C7, C8: 0.33uF, Capacitor_SMD:C_0805_2012Metric_Pad1.18x1.45mm_HandSolder
- removed C12, C3, C35, C43, C6, C9: 100nF, Capacitor_THT:C_Disc_D7.5mm_W5.0mm_P10.00mm
- removed IC1, IC2: CD74HC4050ME4, SamacSys_Parts:SOIC127P600X175-16N
- removed IC15, IC18, IC3, IC4, IC5, IC8: MAX31865AAP+, SamacSys_Parts:SOP65P778X199-20N
- removed J1: RTD1, SamacSys_Parts:1727751
- removed J10, J13, J16, J19, J26, J29: Conn_01x03, Connector_PinHeader_2.54mm:PinHeader_1x03_P2.54mm_Vertical
- removed J11, J12, J14, J15, J17, J18, J20, J25, J27, J28, J30, J9: Conn_01x02, Connector_PinHeader_2.54mm:PinHeader_1x02_P2.54mm_Vertical
- removed J2: RTD2, SamacSys_Parts:1727751
- removed J8: Conn_01x03, Connector_PinSocket_2.54mm:PinSocket_1x03_P2.54mm_Vertical
- removed R2, R20, R3, R36, R4, R60: 430, Resistor_THT:R_Axial_DIN0207_L6.3mm_D2.5mm_P2.54mm_Vertical
- added T1: Conn_01x08, Connector_PinSocket_2.54mm:PinSocket_1x08_P2.54mm_Vertical, F.Cu at (207.6, 77.8)
- added T2: Conn_01x08, Connector_PinSocket_2.54mm:PinSocket_1x08_P2.54mm_Vertical, F.Cu at (200.1, 96.3)
- added T3: Conn_01x08, Connector_PinSocket_2.54mm:PinSocket_1x08_P2.54mm_Vertical, F.Cu at (186.0, 96.4)
- added T4: Conn_01x08, Connector_PinSocket_2.54mm:PinSocket_1x08_P2.54mm_Vertical, F.Cu at (185.4, 133.2)
- added T5: Conn_01x08, Connector_PinSocket_2.54mm:PinSocket_1x08_P2.54mm_Vertical, F.Cu at (200.3, 133.2)
- added T6: Conn_01x08, Connector_PinSocket_2.54mm:PinSocket_1x08_P2.54mm_Vertical, F.Cu at (145.2, 126.1)
- moved R67 108.0 mm to (138.5, 123.0)
- moved IC20 106.8 mm to (131.1, 120.6)
- moved R66 101.7 mm to (138.5, 119.9)
- moved J24 100.6 mm to (181.7, 92.8)
- moved J23 93.7 mm to (178.0, 92.8)
- moved L4 92.6 mm to (205.6, 119.2)
- moved D9 92.6 mm to (219.7, 122.8)
- moved IC13 92.5 mm to (212.8, 129.9)
- moved R64 92.3 mm to (122.8, 116.8)
- moved R65 92.3 mm to (122.9, 123.1)
- moved R68 91.7 mm to (138.4, 126.1)
- moved C30 91.1 mm to (196.4, 123.7)
- moved C29 89.3 mm to (224.2, 117.0)
- moved C28 87.9 mm to (185.6, 123.6)
- moved R69 85.8 mm to (138.4, 129.1)
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Connections:
- Q22 pad 1: Net-(Q22-Pad1) -> +3.3VP
- R63 pad 1: Net-(Q22-Pad1) -> +3.3VP
Routing:
- net GND: track 32.9 -> 41.3 mm
Other:
- board text removed: "2"
- board text removed: "2-3"
- board text removed: "2-4"
- board text removed: "3"
- board text removed: "Ambient Temp"
- board text removed: "CARB Temp"
- board text removed: "Front Temp"
- board text removed: "Left Side Temp"
- board text removed: "Right Side Temp"
- board text removed: "WaterTemp"
